File: electronic/programming.sch (EAGLE design)
At the start: 10 parts

Commit message: add licence hardware
Other:
- note added: "Under Licence CERN OHL version 1.2."
- note removed: "FabKids rev0.2"
Changed lines of the file:
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@@
 <?xml version="1.0" encoding="utf-8"?>
 <!DOCTYPE eagle SYSTEM "eagle.dtd">
-<eagle version="7.7.0">
+<eagle version="9.1.2">
 <drawing>
 <settings>
 <setting alwaysvectorfont="no"/>
+<setting keepoldvectorfont="yes"/>
 <setting verticaltext="up"/>
 </settings>
@@
 <plain>
 <text x="157.48" y="2.54" size="1.778" layer="94" font="vector">Esteban Martin Gimenez</text>
-<text x="132.08" y="-12.7" size="1.778" layer="94" font="vector">FabKids rev0.2</text>
+<text x="167.64" y="-25.4" size="1.778" layer="94" font="vector">Under Licence
+CERN OHL version 1.2.
+</text>
 </plain>
 <instances>
@@
 </schematic>
 </drawing>
+<compatibility>
+<note version="6.3" minversion="6.2.2" severity="warning">
+Since Version 6.2.2 text objects can contain more than one line,
+which will not be processed correctly with this version.
+</note>
+</compatibility>
 </eagle>
